File: hardware/main-control-board/kicad/P0_main_control.kicad_sch (KiCad schematic)
At the start: 34 parts, among them J1 SERVO0, J2 SERVO1, J3 SERVO2, J4 SERVO3, J5 PWR_IN, J6 SERVO_PWR, J7 SWD, Q1 AO4407A, SW1 ESTOP, U1 STM32G474CBT6, U2 MAX485, U3 MAX485, U4 MAX485, U5 MAX485, U6 SI8640, U7 AMS1117-3.3, U8 TPS3823-33

Commit message: fix(hardware): 舵机实为RDS3115 PWM控制，修正P0板4路RS485假设为4路PWM输出并重生成KiCad/EasyEDA工程; docs: 补L1官方规格与RDS3115参数、驱动默认值与官方量程对照(含range_max 100m→30m)、Rviz2可视化，中英同步
Parts:
- removed U2, U3, U4, U5: MAX485, Package_SO:SOIC-8_3.9x4.9mm_P1.27mm, symbol P0lib:MAX485
- added RS1, RS2, RS3, RS4: 220, Resistor_SMD:R_0805_2012Metric, symbol P0lib:R
- J1, J2, J3, J4: footprint Connector_JST:JST_GH_1x04_P1.25mm -> Connector_JST:JST_GH_1x03_P1.25mm; symbol P0lib:CONN4 -> P0lib:CONN3
